File: hardware/kicad-project/diseqc_cntrl_usb.kicad_sch (KiCad schematic)
At the start: 6 parts, among them J5 USB4110-GF-A, U1 FT230XS

Commit message: Corrected TP20 value
Other:
- company: (none) -> M0DMF 
- title: (none) -> DiSEqc Motor Control
Changed lines of the file:
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@@
 	(generator_version "10.0")
 	(paper "A4")
+	(title_block
+		(title "DiSEqc Motor Control")
+		(date "2026-06-09")
+		(rev "0.5-dev")
+		(company "M0DMF ")
+	)
 	(junction
 		(at 111.76 49.53)
