File: hardware/kicad-project/diseqc_cntrl_w5500.kicad_sch (KiCad schematic)
At the start: 30 parts, among them IC6 W5500, J8 RJCSE538101, T1 H1102NL, Y2 25MHZ

Commit message: Corrective changes to power regulation: F1, PS1
Parts:
- C32, C34, C36, C38, C39, C40, C41, R23, R24, R25, R26: My Stock 50 -> (none)
- C35, C37, R21: My Stock 25 -> (none)
- IC6: footprint W5500:QFP50P900X900X160-48N -> diseqc_cntrl:QFP50P900X900X160-48N
- J8: footprint RJCSE538101 -> diseqc_cntrl:RJCSE538101
- R17, R19, R22: My Stock 100 -> (none)
- R18, R20, R27, R28, R29, R30: My Stock 0 -> (none)
- T1: footprint H1102NL:SOIC127P940X597-16N -> diseqc_cntrl:SOIC127P940X597-16N
- Y2: footprint ABLS 25mhz xtal:ABLS25000MHZDFT -> diseqc_cntrl:ABLS25000MHZDFT

Commit message: Starting v0.4 with FT230 fixes; extra TPs
Parts:
- C31: InvenTree Part (none) -> C_4u7_0603
- C32, C34, C36, C38, C39, C40, C41: InvenTree Part (none) -> C_100n_0603; Mouser Part Number 81-GRM39X104K16 -> (none)
- C33: InvenTree Part (none) -> C_10u_0603
- C35, C37: InvenTree Part (none) -> C_18p_0603
- C42: InvenTree Part (none) -> C_22n_0603
- IC6: InvenTree Part (none) -> IC_ETH_100BASETX
- J8: InvenTree Part (none) -> J_ETH_RJ45_SKT_LEDS
- R17, R19: InvenTree Part (none) -> R_10k_0603
- R18: InvenTree Part (none) -> R_12k4_0603_1%
- R20: InvenTree Part (none) -> R_4k7_0603
- R21: InvenTree Part (none) -> R_1M_0603
- R22: InvenTree Part (none) -> R_0r_0603
- R23, R24, R25, R26: InvenTree Part (none) -> R_33r_0603
- R27, R28: InvenTree Part (none) -> R_49r9_0603_1%
- R29, R30: InvenTree Part (none) -> R_470r_0603
- T1: InvenTree Part (none) -> MAG_ETH_10-100_1CH_TH
- Y2: InvenTree Part (none) -> X_25MHZ

Commit message: Added InvenTree part codes
Parts:
- C31: InvenTree (none) -> 76
- C32, C34, C36, C38, C39, C40, C41: InvenTree (none) -> 75
- C33: InvenTree (none) -> 221
- C35, C37: InvenTree (none) -> 66
- C42: InvenTree (none) -> 69
- IC6: InvenTree (none) -> 92
- J8: InvenTree (none) -> 80
- R17, R19: InvenTree (none) -> 106
- R18: InvenTree (none) -> 112; ToleranceRequirement (none) -> <=1%
- R20: InvenTree (none) -> 113
- R21: InvenTree (none) -> 108
- R22: InvenTree (none) -> 104
- R23, R24, R25, R26: InvenTree (none) -> 110
- R27, R28: InvenTree (none) -> 115; ToleranceRequirement (none) -> <=1%
- R29, R30: InvenTree (none) -> 114
- T1: InvenTree (none) -> 120
- Y2: InvenTree (none) -> 83
