File: hardware/kicad-project/diseqc_cntrl.kicad_sch (KiCad schematic)
At the start: 27 parts, among them IC1 TPS560200DBVR, J1 Barrel Jack

Commit message: Adding test points
Parts:
- TP1: value TP_VIN_FUSED -> VIN_FUSED; footprint TestPoint:TestPoint_THTPad_D1.0mm_Drill0.5mm -> ebnx_footprints:TestPoint_THTPad_D1.0mm_Drill0.5mm_annotated; symbol Connector:TestPoint -> ebnx_symbols:TestPoint_Annotated_Silkscreen; now in the parts list
- TP2: value TP_+12V -> PWR_12V; footprint TestPoint:TestPoint_THTPad_D1.0mm_Drill0.5mm -> ebnx_footprints:TestPoint_THTPad_D1.0mm_Drill0.5mm_annotated; symbol Connector:TestPoint -> ebnx_symbols:TestPoint_Annotated_Silkscreen; now in the parts list
- TP3: value TP_+3V3 -> PWR_3V3; footprint TestPoint:TestPoint_THTPad_D1.0mm_Drill0.5mm -> ebnx_footprints:TestPoint_THTPad_D1.0mm_Drill0.5mm_annotated; symbol Connector:TestPoint -> ebnx_symbols:TestPoint_Annotated_Silkscreen; now in the parts list
- TP5: value TP_VIN_PROTECT -> VIN_PROTECT; footprint TestPoint:TestPoint_THTPad_D1.0mm_Drill0.5mm -> ebnx_footprints:TestPoint_THTPad_D1.0mm_Drill0.5mm_annotated; symbol Connector:TestPoint -> ebnx_symbols:TestPoint_Annotated_Silkscreen; now in the parts list
Changed lines of the file:
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@@
 	)
 	(symbol
-		(lib_id "Connector:TestPoint")
+		(lib_id "ebnx_symbols:TestPoint_Annotated_Silkscreen")
 		(at 245.11 99.06 270)
 		(unit 1)
 		(body_style 1)
 		(exclude_from_sim no)
-		(in_bom no)
+		(in_bom yes)
 		(on_board yes)
 		(in_pos_files yes)
@@
 			)
 		)
-		(property "Value" "TP_VIN_FUSED"
+		(property "Value" "VIN_FUSED"
 			(at 250.19 100.3299 90)
 			(show_name no)
@@
 			)
 		)
-		(property "Footprint" "TestPoint:TestPoint_THTPad_D1.0mm_Drill0.5mm"
+		(property "Footprint" "ebnx_footprints:TestPoint_THTPad_D1.0mm_Drill0.5mm_annotated"
 			(at 245.11 104.14 0)
 			(hide yes)
@@
 	)
 	(symbol
-		(lib_id "Connector:TestPoint")
+		(lib_id "ebnx_symbols:TestPoint_Annotated_Silkscreen")
 		(at 245.11 111.76 270)
 		(unit 1)
 		(body_style 1)
 		(exclude_from_sim no)
-		(in_bom no)
+		(in_bom yes)
 		(on_board yes)
 		(in_pos_files yes)
@@
 			)
 		)
-		(property "Value" "TP_+3V3"
+		(property "Value" "PWR_3V3"
 			(at 250.19 113.0299 90)
 			(show_name no)
@@
 			)
 		)
-		(property "Footprint" "TestPoint:TestPoint_THTPad_D1.0mm_Drill0.5mm"
+		(property "Footprint" "ebnx_footprints:TestPoint_THTPad_D1.0mm_Drill0.5mm_annotated"
 			(at 245.11 116.84 0)
 			(hide yes)
@@
 	)
 	(symbol
-		(lib_id "Connector:TestPoint")
+		(lib_id "ebnx_symbols:TestPoint_Annotated_Silkscreen")
 		(at 245.11 105.41 270)
 		(unit 1)
 		(body_style 1)
 		(exclude_from_sim no)
-		(in_bom no)
+		(in_bom yes)
 		(on_board yes)
 		(in_pos_files yes)
@@
 			)
 		)
-		(property "Value" "TP_+12V"
+		(property "Value" "PWR_12V"
 			(at 250.19 106.6799 90)
 			(show_name no)
@@
 			)
 		)
-		(property "Footprint" "TestPoint:TestPoint_THTPad_D1.0mm_Drill0.5mm"
+		(property "Footprint" "ebnx_footprints:TestPoint_THTPad_D1.0mm_Drill0.5mm_annotated"
 			(at 245.11 110.49 0)
 			(hide yes)
@@
 	)
 	(symbol
-		(lib_id "Connector:TestPoint")
+		(lib_id "ebnx_symbols:TestPoint_Annotated_Silkscreen")
 		(at 245.11 124.46 270)
 		(unit 1)
 		(body_style 1)
 		(exclude_from_sim no)
-		(in_bom no)
+		(in_bom yes)
 		(on_board yes)
 		(in_pos_files yes)
@@
 			)
 		)
-		(property "Value" "TP_VIN_PROTECT"
+		(property "Value" "VIN_PROTECT"
 			(at 250.19 125.7299 90)
 			(show_name no)
@@
 			)
 		)
-		(property "Footprint" "TestPoint:TestPoint_THTPad_D1.0mm_Drill0.5mm"
+		(property "Footprint" "ebnx_footprints:TestPoint_THTPad_D1.0mm_Drill0.5mm_annotated"
 			(at 245.11 129.54 0)
 			(hide yes)
