File: hardware/kicad-project/diseqc_cntrl_mcu.kicad_sch (KiCad schematic)
At the start: 40 parts, among them IC2 STM32F407VGT6, IC3 FM24CL16B-GTR, IC4 USBLC6-2P6, J2 Conn_01x04_Pin, J3 USB4110-GF-A, J4 TC2050, J9 Conn_01x04_Pin, SW1 Reset, Y1 8MHZ

Commit message: Renumbered/annotated
Parts:
- renumbered C6 to C13, C8 to C14, C7 to C15, C9 to C16, C10 to C17, C11 to C18, C12 to C19, C13 to C20, C14 to C21, C16 to C22, C17 to C23, C18 to C24, C19 to C25, C20 to C26, C15 to C27, IC2 to IC3, IC3 to IC4, IC4 to IC5, J9 to J2, J2 to J3, J3 to J4, J4 to J5, R12 to R10, R13 to R11, R14 to R12, R15 to R13, R16 to R14, R7 to R5, R8 to R6, R9 to R7, R10 to R8, R11 to R9, TP25 to TP8, TP6 to TP9

Commit message: Replaced 10k pull-up on NRST
Parts:
- added R38: 10k, Resistor_SMD:R_0603_1608Metric, symbol #InvenTree:R_10k_0603
Connections:
- net +3V3: now also R38.1
- net NRST: now also R38.2
Changed lines of the file:
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@@
 	(wire
 		(pts
+			(xy 58.42 55.88) (xy 58.42 53.34)
+		)
+		(stroke
+			(width 0)
+			(type default)
+		)
+	)
+	(wire
+		(pts
 			(xy 234.95 146.05) (xy 228.6 146.05)
 		)
@@
 		)
 	)
+	(wire
+		(pts
+			(xy 58.42 63.5) (xy 58.42 72.39)
+		)
+		(stroke
+			(width 0)
+			(type default)
+		)
+	)
 	(bus
 		(pts
@@
 	(wire
 		(pts
+			(xy 58.42 72.39) (xy 68.58 72.39)
+		)
+		(stroke
+			(width 0)
+			(type default)
+		)
+	)
+	(wire
+		(pts
 			(xy 68.58 114.3) (xy 53.34 114.3)
 		)
@@
 	)
 	(symbol
+		(lib_id "#InvenTree:R_10k_0603")
+		(at 58.42 59.69 0)
+		(unit 1)
+		(body_style 1)
+		(exclude_from_sim no)
+		(in_bom yes)
+		(on_board yes)
+		(in_pos_files yes)
+		(dnp no)
+		(fields_autoplaced yes)
+		(property "Reference" "R38"
+			(at 60.96 58.4199 0)
+			(show_name no)
+			(do_not_autoplace no)
+			(effects
+				(font
+					(size 1.27 1.27)
+				)
+				(justify left)
+			)
+		)
+		(property "Value" "10k"
+			(at 60.96 60.9599 0)
+			(show_name no)
+			(do_not_autoplace no)
+			(effects
+				(font
+					(size 1.27 1.27)
+				)
+				(justify left)
+			)
+		)
+		(property "Footprint" "Resistor_SMD:R_0603_1608Metric"
+			(at 56.642 59.69 90)
+			(hide yes)
+			(show_name no)
+			(do_not_autoplace no)
+			(effects
+				(font
+					(size 1.27 1.27)
+				)
+			)
+		)
+		(property "Datasheet" ""
+			(at 58.42 59.69 0)
+			(hide yes)
+			(show_name no)
+			(do_not_autoplace no)
+			(effects
+				(font
+					(size 1.27 1.27)
+				)
+			)
+		)
+		(property "Description" "10k Resistor"
+			(at 58.42 59.69 0)
+			(hide yes)
+			(show_name no)
+			(do_not_autoplace no)
+			(effects
+				(font
+					(size 1.27 1.27)
+				)
+			)
+		)
+		(property "InvenTree" "106"
+			(at 58.42 59.69 0)
+			(hide yes)
+			(show_name no)
+			(do_not_autoplace no)
+			(effects
+				(font
+					(size 1.27 1.27)
+				)
+			)
+		)
+		(property "Part URL" "https://inventree.ebnx.net/web/part/106/"
+			(at 58.42 59.69 0)
+			(hide yes)
+			(show_name no)
+			(do_not_autoplace no)
+			(effects
+				(font
+					(size 1.27 1.27)
+				)
+			)
+		)
+		(pin "1"
+		)
+		(pin "2"
+		)
+		(instances
+			(project "diseqc_cntrl"
+				(path "/82a905d8-f1d7-4995-9c16-94cf3cdcaad9/65fcf1a0-d0f2-4bf0-9977-67dd9f84afa5"
+					(reference "R38")
+					(unit 1)
+				)
+			)
+		)
+	)
+	(symbol
 		(lib_id "diseqc_cntrl:C")
 		(at 38.1 33.02 0)
@@
 					(unit 1)
 				)
+			)
+		)
+	)
+	(symbol
+		(lib_id "diseqc_cntrl:+3V3")
+		(at 58.42 53.34 0)
+		(unit 1)
+		(body_style 1)
+		(exclude_from_sim no)
+		(in_bom yes)
+		(on_board yes)
+		(in_pos_files yes)
+		(dnp no)
+		(property "Reference" "#PWR073"
+			(at 58.42 57.15 0)
+			(hide yes)
+			(show_name no)
+			(do_not_autoplace no)
+			(effects
+				(font
+					(size 1.27 1.27)
+				)
+			)
+		)
+		(property "Value" "+3V3"
+			(at 58.166 49.53 0)
+			(show_name no)
+			(do_not_autoplace no)
+			(effects
+				(font
+					(size 1.27 1.27)
+				)
+			)
+		)
+		(property "Footprint" ""
+			(at 58.42 53.34 0)
+			(hide yes)
+			(show_name no)
+			(do_not_autoplace no)
+			(effects
+				(font
+					(size 1.27 1.27)
+				)
+			)
+		)
+		(property "Datasheet" ""
+			(at 58.42 53.34 0)
+			(hide yes)
+			(show_name no)
+			(do_not_autoplace no)
+			(effects
+				(font
+					(size 1.27 1.27)
+				)
+			)
+		)
+		(property "Description" "Power symbol creates a global label with name \"+3V3\""
+			(at 58.42 53.34 0)
+			(hide yes)
+			(show_name no)
+			(do_not_autoplace no)
+			(effects
+				(font
+					(size 1.27 1.27)
+				)
+			)
+		)
+		(pin "1"
+		)
+		(instances
+			(project "diseqc_cntrl"
+				(path "/82a905d8-f1d7-4995-9c16-94cf3cdcaad9/65fcf1a0-d0f2-4bf0-9977-67dd9f84afa5"
+					(reference "#PWR073")
+					(unit 1)
+				)

Commit message: Decreased VBUS_SENSE (R8) to 1k
Parts:
- J2: now not fitted; now left out of the parts list
- R8: value 100k -> 1k; symbol diseqc_cntrl:R -> #InvenTree:R_1k_0603_5%; InvenTree 105 -> 176; InvenTree Part R_100k_0603 -> (none); Mouser Part Number 603-RC0603JR-07100KL -> (none); Part URL (none) -> https://inventree.ebnx.net/web/part/176/; Tolerance (none) -> 5%
Changed lines of the file:
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@@
 		(body_style 1)
 		(exclude_from_sim no)
-		(in_bom yes)
+		(in_bom no)
 		(on_board yes)
 		(in_pos_files yes)
-		(dnp no)
+		(dnp yes)
 		(fields_autoplaced yes)
 		(property "Reference" "J2"
@@
 	)
 	(symbol
-		(lib_id "diseqc_cntrl:R")
+		(lib_id "#InvenTree:R_1k_0603_5%")
 		(at 165.1 76.2 90)
 		(unit 1)
@@
 		(dnp no)
 		(property "Reference" "R8"
-			(at 165.1 71.12 90)
+			(at 165.1 72.136 90)
 			(show_name no)
 			(do_not_autoplace no)
@@
 			)
 		)
-		(property "Value" "100k"
-			(at 165.1 73.66 90)
+		(property "Value" "1k"
+			(at 165.1 73.914 90)
 			(show_name no)
 			(do_not_autoplace no)
@@
 			)
 		)
-		(property "Datasheet" "https://www.mouser.com/catalog/specsheets/YAGEO_PYu_RC_Group_51_RoHS_L_12.pdf"
+		(property "Datasheet" ""
 			(at 165.1 76.2 0)
 			(hide yes)
@@
 			)
 		)
-		(property "Mouser Part Number" "603-RC0603JR-07100KL"
+		(property "Mouser Part Number" ""
 			(at 165.1 76.2 0)
 			(hide yes)
@@
 			)
 		)
-		(property "InvenTree Part" "R_100k_0603"
+		(property "InvenTree Part" ""
 			(at 165.1 76.2 90)
 			(hide yes)
@@
 			)
 		)
-		(property "Tolerance" ""
-			(at 165.1 76.2 90)
+		(property "Tolerance" "5%"
+			(at 165.1 76.2 0)
 			(hide yes)
 			(show_name no)
@@
 			)
 		)
-		(property "InvenTree" "105"
-			(at 165.1 76.2 90)
+		(property "InvenTree" "176"
+			(at 165.1 76.2 0)
+			(hide yes)
+			(show_name no)
+			(do_not_autoplace no)
+			(effects
+				(font
+					(size 1.27 1.27)
+				)
+			)
+		)
+		(property "Part URL" "https://inventree.ebnx.net/web/part/176/"
+			(at 165.1 76.2 0)
 			(hide yes)
 			(show_name no)

Commit message: Added LNB Fault pull-up and LED
Parts:
- added LED1: Red, LED_SMD:LED_0603_1608Metric, symbol #InvenTree:LED_Red_0603
- added R39: 10k, Resistor_SMD:R_0603_1608Metric, symbol #InvenTree:R_10k_0603
- added R40: 1k5, Resistor_SMD:R_0603_1608Metric, symbol #InvenTree:R_1k5_0603
- added TP12: LNB_FAULT, ebnx_footprints:TestPoint_THTPad_D1.0mm_Drill0.5mm_annotated, symbol ebnx_symbols:TestPoint_Annotated_Silkscreen
- LED2: renamed from D3; footprint LED_SMD:LED_0603_1608Metric_Pad1.05x0.95mm_HandSolder -> LED_SMD:LED_0603_1608Metric; symbol diseqc_cntrl:LED_Small -> #InvenTree:LED_Green_0603; Part URL (none) -> https://inventree.ebnx.net/web/part/99/
Connections:
- net GND: now also R40.1
- net LNB_FLT renamed SIG_LNB_FLT
- net SIG_LNB_FLT: now also R39.1, TP12.1
- new net: LED1.1 (K), R40.2
- new net LNBH26PQR/LNB_FLT: LED1.2 (A), R39.2
Other:
- moved on the sheet: LED2

Commit message: Updated Vreg output caps to match datasheet
Parts:
- removed C13: 4.7u, Capacitor_SMD:C_0603_1608Metric, symbol diseqc_cntrl:C_Small
Changed lines of the file:
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@@
-	(symbol
-		(lib_id "diseqc_cntrl:C_Small")
-		(at 16.51 167.64 0)
-		(unit 1)
-		(body_style 1)
-		(exclude_from_sim no)
-		(in_bom yes)
-		(on_board yes)
-		(in_pos_files yes)
-		(dnp no)
-		(property "Reference" "C13"
-			(at 19.05 166.37 0)
-			(show_name no)
-			(do_not_autoplace no)
-			(effects
-				(font
-					(size 1.27 1.27)
-				)
-				(justify left)
-			)
-		)
-		(property "Value" "4.7u"
-			(at 19.05 168.91 0)
-			(show_name no)
-			(do_not_autoplace no)
-			(effects
-				(font
-					(size 1.27 1.27)
-				)
-				(justify left)
-			)
-		)
-		(property "Footprint" "Capacitor_SMD:C_0603_1608Metric"
-			(at 16.51 167.64 0)
-			(hide yes)
-			(show_name no)
-			(do_not_autoplace no)
-			(effects
-				(font
-					(size 1.27 1.27)
-				)
-			)
-		)
-		(property "Datasheet" "https://www.mouser.com/catalog/specsheets/taiyo%20yuden_12132018_mlcc11_hq_e.pdf"
-			(at 16.51 167.64 0)
-			(hide yes)
-			(show_name no)
-			(do_not_autoplace no)
-			(effects
-				(font
-					(size 1.27 1.27)
-				)
-			)
-		)
-		(property "Description" ""
-			(at 16.51 167.64 0)
-			(show_name no)
-			(do_not_autoplace no)
-			(effects
-				(font
-					(size 1.27 1.27)
-				)
-			)
-		)
-		(property "LCSC Part #" "C19666"
-			(at 16.51 167.64 0)
-			(hide yes)
-			(show_name no)
-			(do_not_autoplace no)
-			(effects
-				(font
-					(size 1.27 1.27)
-				)
-			)
-		)
-		(property "Maufacturer_Part_Number" ""
-			(at 16.51 167.64 0)
-			(hide yes)
-			(show_name no)
-			(do_not_autoplace no)
-			(effects
-				(font
-					(size 1.27 1.27)
-				)
-			)
-		)
-		(property "Manufacturer_Part_Code" ""
-			(at 16.51 167.64 0)
-			(hide yes)
-			(show_name no)
-			(do_not_autoplace no)
-			(effects
-				(font
-					(size 1.27 1.27)
-				)
-			)
-		)
-		(property "Mouser_Part_Number" ""
-			(at 16.51 167.64 0)
-			(hide yes)
-			(show_name no)
-			(do_not_autoplace no)
-			(effects
-				(font
-					(size 1.27 1.27)
-				)
-			)
-		)
-		(property "Mouser Part Number" "963-JMK107BJ475KAHT"
-			(at 16.51 167.64 0)
-			(hide yes)
-			(show_name no)
-			(do_not_autoplace no)
-			(effects
-				(font
-					(size 1.27 1.27)
-				)
-			)
-		)
-		(property "InvenTree Part" "C_4u7_0603"
-			(at 16.51 167.64 0)
-			(hide yes)
-			(show_name no)
-			(do_not_autoplace no)
-			(effects
-				(font
-					(size 1.27 1.27)
-				)
-			)
-		)
-		(property "KLC_S4.2_3V3OUT" ""
-			(at 16.51 167.64 0)
-			(hide yes)
-			(show_name no)
-			(do_not_autoplace no)
-			(effects
-				(font
-					(size 1.27 1.27)
-				)
-			)
-		)
-		(property "KLC_S4.2_VCC" ""
-			(at 16.51 167.64 0)
-			(hide yes)
-			(show_name no)
-			(do_not_autoplace no)
-			(effects
-				(font
-					(size 1.27 1.27)
-				)
-			)
-		)
-		(property "Tolerance" ""
-			(at 16.51 167.64 0)
-			(hide yes)
-			(show_name no)
-			(do_not_autoplace no)
-			(effects
-				(font
-					(size 1.27 1.27)
-				)
-			)
-		)
-		(property "InvenTree" "76"
-			(at 16.51 167.64 0)
-			(hide yes)
-			(show_name no)
-			(do_not_autoplace no)
-			(effects
-				(font
-					(size 1.27 1.27)
-				)
-			)
-		)
-		(pin "1"
-		)
-		(pin "2"
-		)
-		(instances
-			(project "diseqc_cntrl"
-				(path "/82a905d8-f1d7-4995-9c16-94cf3cdcaad9/65fcf1a0-d0f2-4bf0-9977-67dd9f84afa5"
-					(reference "C13")
-					(unit 1)
-				)
-			)
-		)
-	)
 	(symbol
 		(lib_id "diseqc_cntrl:C_Small")

Commit message: Add fiducials
Parts:
- LED2: renamed from LED1; InvenTree Part (none) -> LED_Red_0603
- renumbered C14 to C18, C15 to C19, C16 to C20, C17 to C21, C18 to C22, C19 to C23, C20 to C24, C21 to C25, C22 to C26, C23 to C27, C24 to C28, C25 to C29, C26 to C30, C27 to C31, LED2 to LED1, R9 to R10, R10 to R11, R11 to R12, R12 to R13, R40 to R14, R39 to R15, R13 to R16, R14 to R17, R38 to R6, R6 to R7, R7 to R8, R8 to R9, TP12 to TP10

Commit message: Upgraded power supplies
Parts:
- JP2: footprint TestPoint:TestPoint_2Pads_Pitch2.54mm_Drill0.8mm -> Connector_PinHeader_2.54mm:PinHeader_1x02_P2.54mm_Vertical
Changed lines of the file:
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@@
 	)
 	(junction
-		(at 77.47 162.56)
-		(diameter 0)
-		(color 0 0 0 0)
-	)
-	(junction
 		(at 213.36 34.29)
 		(diameter 0)
@@
 	)
 	(junction
-		(at 77.47 172.72)
+		(at 55.88 172.72)
 		(diameter 0)
 		(color 0 0 0 0)
 	)
 	(junction
-		(at 55.88 172.72)
+		(at 77.47 172.72)
 		(diameter 0)
 		(color 0 0 0 0)
@@
 	)
 	(junction
-		(at 25.4 162.56)
-		(diameter 0)
-		(color 0 0 0 0)
-	)
-	(junction
 		(at 185.42 78.74)
 		(diameter 0)
@@
 	)
 	(junction
-		(at 25.4 172.72)
-		(diameter 0)
-		(color 0 0 0 0)
-	)
-	(junction
 		(at 67.31 172.72)
 		(diameter 0)
@@
 	)
 	(junction
+		(at 77.47 162.56)
+		(diameter 0)
+		(color 0 0 0 0)
+	)
+	(junction
 		(at 142.24 166.37)
 		(diameter 0)
@@
 	(wire
 		(pts
-			(xy 16.51 162.56) (xy 77.47 162.56)
+			(xy 25.4 162.56) (xy 77.47 162.56)
 		)
 		(stroke
@@
 	(wire
 		(pts
-			(xy 16.51 172.72) (xy 77.47 172.72)
+			(xy 25.4 172.72) (xy 77.47 172.72)
 		)
 		(stroke
@@
 	(wire
 		(pts
-			(xy 16.51 162.56) (xy 16.51 165.1)
-		)
-		(stroke
-			(width 0)
-			(type default)
-		)
-	)
-	(wire
-		(pts
 			(xy 168.91 76.2) (xy 170.18 76.2)
 		)
@@
 	(wire
 		(pts
-			(xy 16.51 170.18) (xy 16.51 172.72)
-		)
-		(stroke
-			(width 0)
-			(type default)
-		)
-	)
-	(wire
-		(pts
 			(xy 38.1 26.67) (xy 38.1 29.21)
 		)
@@
 			)
 		)
-		(property "Footprint" "TestPoint:TestPoint_2Pads_Pitch2.54mm_Drill0.8mm"
+		(property "Footprint" "Connector_PinHeader_2.54mm:PinHeader_1x02_P2.54mm_Vertical"
 			(at 191.77 30.48 0)
 			(hide yes)

Commit message: Corrected thermal/EMC issues
Parts:
- C20, C22, C24, C25, C26, C27: LCSC Part # C1525 -> (none)
- JP2: InvenTree (none) -> 77
Connections:
- net +3.3VA: now also IC3.21 (VREF+)
- no-connect marks 59 -> 58
Changed lines of the file:
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@@
 	)
 	(no_connect
-		(at 68.58 127)
-	)
-	(no_connect
 		(at 140.97 50.8)
 	)
@@
 	(wire
 		(pts
+			(xy 66.04 138.43) (xy 68.58 138.43)
+		)
+		(stroke
+			(width 0)
+			(type default)
+		)
+	)
+	(wire
+		(pts
 			(xy 134.62 30.48) (xy 137.16 30.48)
 		)
@@
 	(wire
 		(pts
+			(xy 68.58 138.43) (xy 68.58 127)
+		)
+		(stroke
+			(width 0)
+			(type default)
+		)
+	)
+	(wire
+		(pts
 			(xy 93.98 152.4) (xy 93.98 147.32)
 		)
@@
 			)
 		)
-		(property "LCSC Part #" "C1525"
+		(property "LCSC Part #" ""
 			(at 25.4 167.64 0)
 			(hide yes)
@@
 			)
 		)
-		(property "LCSC Part #" "C1525"
+		(property "LCSC Part #" ""
 			(at 35.56 167.64 0)
 			(hide yes)
@@
 			)
 		)
-		(property "LCSC Part #" "C1525"
+		(property "LCSC Part #" ""
 			(at 45.72 167.64 0)
 			(hide yes)
@@
 			)
 		)
-		(property "LCSC Part #" "C1525"
+		(property "LCSC Part #" ""
 			(at 55.88 167.64 0)
 			(hide yes)
@@
 			)
 		)
-		(property "LCSC Part #" "C1525"
+		(property "LCSC Part #" ""
 			(at 67.31 167.64 0)
 			(hide yes)
@@
 			)
 		)
+		(property "InvenTree" "77"
+			(at 191.77 30.48 90)
+			(hide yes)
+			(show_name no)
+			(do_not_autoplace no)
+			(effects
+				(font
+					(size 0.762 0.762)
+				)
+			)
+		)
 		(pin "1"
 		)
@@
 			)
 		)
-		(property "LCSC Part #" "C1525"
+		(property "LCSC Part #" ""
 			(at 77.47 167.64 0)
 			(hide yes)
@@
 					(unit 1)
 				)
+			)
+		)
+	)
+	(symbol
+		(lib_id "power:+3.3VA")
+		(at 66.04 138.43 0)
+		(unit 1)
+		(body_style 1)
+		(exclude_from_sim no)
+		(in_bom yes)
+		(on_board yes)
+		(in_pos_files yes)
+		(dnp no)
+		(fields_autoplaced yes)
+		(property "Reference" "#PWR077"
+			(at 66.04 142.24 0)
+			(hide yes)
+			(show_name no)
+			(do_not_autoplace no)
+			(effects
+				(font
+					(size 1.27 1.27)
+				)
+			)
+		)
+		(property "Value" "+3.3VA"
+			(at 66.04 133.35 0)
+			(show_name no)
+			(do_not_autoplace no)
+			(effects
+				(font
+					(size 1.27 1.27)
+				)
+			)
+		)
+		(property "Footprint" ""
+			(at 66.04 138.43 0)
+			(hide yes)
+			(show_name no)
+			(do_not_autoplace no)
+			(effects
+				(font
+					(size 1.27 1.27)
+				)
+			)
+		)
+		(property "Datasheet" ""
+			(at 66.04 138.43 0)
+			(hide yes)
+			(show_name no)
+			(do_not_autoplace no)
+			(effects
+				(font
+					(size 1.27 1.27)
+				)
+			)
+		)
+		(property "Description" "Power symbol creates a global label with name \"+3.3VA\""
+			(at 66.04 138.43 0)
+			(hide yes)
+			(show_name no)
+			(do_not_autoplace no)
+			(effects
+				(font
+					(size 1.27 1.27)
+				)
+			)
+		)
+		(pin "1"
+		)
+		(instances
+			(project "diseqc_cntrl"
+				(path "/82a905d8-f1d7-4995-9c16-94cf3cdcaad9/65fcf1a0-d0f2-4bf0-9977-67dd9f84afa5"
+					(reference "#PWR077")
+					(unit 1)
+				)
